File: CM5.kicad_sch (KiCad schematic)
At the start: 37 parts, among them CN10 BM04B-SRSS-TB, CN4 10164227-1001A1RLF, CN5 10164227-1001A1RLF, CN6 1.25-6PWT, CN7 B2B-PH-K-S, SW1 TS-1088, U1 DSHP05TSGER_2, U12 RT9742GGJ5, U20 MAX98357AETE+T

Commit message: 1
Parts:
- removed R4, R5: 0603WAF5101T5E, EasyEDA:R0603, symbol JLSC:0603WAF5101T5E
- removed SW1: TS-1088, EasyEDA:SW-SMD_L3.9-W3.0-P4.45, symbol JLSC:TS-1088-AR02016
- removed TP9: CM VBUS Test Point, TestPoint:TestPoint_Pad_D1.0mm, symbol Connector:TestPoint
- removed USBC1: TYPE-C-31-M-12, EasyEDA:USB-C_SMD-TYPE-C-31-M-12_1, symbol JLSC:TYPE-C-31-M-12
- added CN12: HD219F-3D05200, EasyEDA:HDMI-SMD_HD219F-3D05200, symbol JLSC:HD219F-3D05200
Connections:
- net 3.3V_CM5: now also FPC1.1, FPC2.1; no longer FPC1.22, FPC2.22, R22.2
- net 5V: now also CN12.18 (+5V)
- net CAM_GPIO0: now also FPC1.6; no longer FPC1.17
- net CAM_GPIO1: now also FPC1.5; no longer FPC1.18
- net DPHY0_C_N: now also FPC1.15; no longer FPC1.8
- net DPHY0_C_P: now also FPC1.14; no longer FPC1.9
- net DPHY0_D0_N: now also FPC1.21; no longer FPC1.2
- net DPHY0_D0_P: now also FPC1.20; no longer FPC1.3
- net DPHY0_D1_N: now also FPC1.18; no longer FPC1.5
- net DPHY0_D1_P: now also FPC1.17; no longer FPC1.6
- net DPHY0_D2_N: now also FPC1.12; no longer FPC1.11
- net DPHY0_D2_P: now also FPC1.11; no longer FPC1.12
- net DPHY0_D3_N: now also FPC1.9; no longer FPC1.14
- net DPHY0_D3_P: now also FPC1.8; no longer FPC1.15
- net DPHY1_C_N: now also FPC2.15; no longer FPC2.8
- net DPHY1_C_P: now also FPC2.14; no longer FPC2.9
- net DPHY1_D0_N: now also FPC2.21; no longer FPC2.2
- net DPHY1_D0_P: now also FPC2.20; no longer FPC2.3
- net DPHY1_D1_N: now also FPC2.18; no longer FPC2.5
- net DPHY1_D1_P: now also FPC2.17; no longer FPC2.6
- net DPHY1_D2_N: now also FPC2.12; no longer FPC2.11
- net DPHY1_D2_P: now also FPC2.11; no longer FPC2.12
- net DPHY1_D3_N: now also FPC2.9; no longer FPC2.14
- net DPHY1_D3_P: now also FPC2.8; no longer FPC2.15
- net GND: now also FPC1.22, FPC2.22, R22.1, CN12.11 (TMDSClock+), CN12.17 (Utility), CN12.2 (TMDSDATA2+), CN12.20 (EH), CN12.21 (EH), CN12.22 (EH), CN12.23 (EH), CN12.5 (TMDSDATA1+), CN12.8 (TMDSDATA0+); no longer FPC1.1, FPC2.1, FPC2.13
- net SCL0: now also FPC1.3; no longer FPC1.20
- net SCL1: now also FPC2.3; no longer FPC2.20
- net SDA0: now also FPC1.2; no longer FPC1.21
- net SDA1: now also FPC2.2; no longer FPC2.21
- net HDMI1_HOTPLUG: now reaches CN5.43
- net HDMI1_HOTPLUG: now also CN12.19 (HotPlugDetect)
- net HDMI1_SDA: now reaches CN5.45
- net HDMI1_SDA: now also CN12.16 (SDA)
- net HDMI1_D2_P: now reaches CN5.46
- net HDMI1_D2_P: now also CN12.1 (TMDSDATA2Shield)
- net HDMI1_SCL: now reaches CN5.47
- net HDMI1_SCL: now also CN12.15 (SCL)
- net HDMI1_D2_N: now reaches CN5.48
- net HDMI1_D2_N: now also CN12.3 (TMDSDATA2-)
- net HDMI1_CEC: now reaches CN5.49
- net HDMI1_CEC: now also FPC2.13, CN12.13 (DDC/CECGND)
- net HDMI0_CEC: now reaches CN5.51
- net HDMI1_D1_P: now reaches CN5.52
- net HDMI1_D1_P: now also CN12.4 (TMDSDATA1Shield)
- net HDMI0_HOTPLUG: now reaches CN5.53
- net HDMI1_D1_N: now reaches CN5.54
- net HDMI1_D1_N: now also CN12.6 (TMDSDATA1-)
- net HDMI1_D0_P: now reaches CN5.58
- net HDMI1_D0_P: now also CN12.7 (TMDSDATA0Shield)
- net HDMI1_D0_N: now reaches CN5.60
- net HDMI1_D0_N: now also CN12.9 (TMDSDATA0-)
- net HDMI1_CK_P: now reaches CN5.64
- net HDMI1_CK_P: now also CN12.10 (TMDSClockShield)
- net HDMI1_CK_N: now reaches CN5.66
- net HDMI1_CK_N: now also CN12.12 (TMDSClock-)
- net PCIE_CLK_N: no longer names the net of CN5.12
- net PCIE_CLK_P: no longer names the net of CN5.10
- net PCIE_PWR_EN: no longer names the net of CN5.6
- net PCIE_RX_N: no longer names the net of CN5.18
- net PCIE_RX_P: no longer names the net of CN5.16
- net PCIE_TX_N: no longer names the net of CN5.24
- net PCIE_TX_P: no longer names the net of CN5.22
- net PCIE_nCLKREQ: no longer names the net of CN5.2
- net PCIE_nRST: no longer names the net of CN5.9
- net PCIE_nWAKE: no longer names the net of CN5.4
- new net: FPC2.6, R22.2
- no-connect marks 87 -> 82
Other:
- note added: "HDMI"
- note removed: "Power Switch"
- note removed: "Type-C Connector"
- moved on the sheet: CN6, FPC1, FPC2, H10, H11, H12, H9, LED3, R22, R8

Commit message: micro hdmi eklendi
Parts:
- removed C32: 100uF, EasyEDA:CAP-SMD_BD6.3-L6.6-W6.6-LS7.2-R-RD, symbol JLSC:RVT1E101M0607
- removed CN12: HD219F-3D05200, EasyEDA:HDMI-SMD_HD219F-3D05200, symbol JLSC:HD219F-3D05200
- added C1, C2: 100nF, EasyEDA:C0603, symbol JLSC:CC0603KRX7R9BB104
- added C3: 100uF, EasyEDA:CAP-SMD_BD6.3-L6.6-W6.6-LS7.2-R-RD, symbol JLSC:RVT1E101M0607
- added U11: RT9742SNGV_C3235509, EasyEDA:SOT-23-3_L2.9-W1.6-P1.90-LS2.8-BR, symbol JLSC:RT9742SNGV_C3235509
- added USB3: HDMI-101L, EasyEDA:HDMI-SMD_HDMI-101L, symbol JLSC:HDMI-101L
Connections:
- net 3.3V_CM5: now also R22.1
- net 5V: now also C2.2, C3.1, U11.1 (VIN)
- net GND: now also FPC2.13, C1.2, C2.1, C3.2, U11.3 (GND), USB3.10 (TMDS_DATA0_SHIELD), USB3.13 (TMDS_CLOCK_SHIELD), USB3.16 (DDC/CEC_GND), USB3.2 (UTILITY), USB3.20 (SHIELD), USB3.4 (TMDS_DATA2_SHIELD), USB3.7 (TMDS_DATA1_SHIELD); no longer R22.1
- net HDMI1_CEC: now also USB3.15 (CEC); no longer FPC2.13
- net HDMI1_CK_N: now also USB3.14 (TMDS_CLOCK-)
- net HDMI1_CK_P: now also USB3.12 (TMDS_CLOCK+)
- net HDMI1_D0_N: now also USB3.11 (TMDS_DATA0-)
- net HDMI1_D0_P: now also USB3.9 (TMDS_DATA0+)
- net HDMI1_D1_N: now also USB3.8 (TMDS_DATA1-)
- net HDMI1_D1_P: now also USB3.6 (TMDS_DATA1+)
- net HDMI1_D2_N: now also USB3.5 (TMDS_DATA2-)
- net HDMI1_D2_P: now also USB3.3 (TMDS_DATA2+)
- net HDMI1_HOTPLUG: now also USB3.1 (HOT_PLUG_DET)
- net HDMI1_SCL: now also USB3.17 (SCL)
- net HDMI1_SDA: now also USB3.18 (SDA)
- net HDMI0_CEC: no longer names the net of CN5.51
- net HDMI0_HOTPLUG: no longer names the net of CN5.53
- net USB2_N: no longer names the net of CN5.3
- net USB2_P: no longer names the net of CN5.5
- new net HDMI_5v: C1.1, U11.2 (VOUT), USB3.19 (+5V)
- no-connect marks 82 -> 86
