File: Orbit Mini Mainboard.kicad_pcb (KiCad board)
At the start: 6 copper layers, 80 x 105 mm, 171 parts, among them CN1 A1251WV-8P, CN10 BM04B-SRSS-TB, CN11 XH-2A, CN12 HD219F-3D05200, CN2 B2B-PH-K-S, CN3 PH-3A_C2908624, CN4 10164227-1001A1RLF, CN5 10164227-1001A1RLF, CN6 1.25-6PWT, CN7 B2B-PH-K-S, CN8 XH-2A, CN9 XH-2A, U1 DSHP05TSGER_2, U10 DRV8848PWPR, U12 RT9742GGJ5, U16 LMR50410XDBVR, U17 LMR50410XDBVR, U18 2.00mm-4P-JST, U2 2.00mm-4P-JST, U20 MAX98357AETE+T, U21 TCA9534PWR, U22 PZ2.54-2*4, U3 BQ25792RQMR, U4 INA228AIDGSR, U5 TPS56A37RPAR, U6 IHLP3232DZER3R3M01, U7 ESP32-S3-WROOM-1, U8 LSM6DSOXTR, U9 SN74LVC1G32DBVR

Commit message: micro hdmi eklendi
Parts:
- removed C32: 100uF, EasyEDA:CAP-SMD_BD6.3-L6.6-W6.6-LS7.2-R-RD
- removed CN12: HD219F-3D05200, EasyEDA:HDMI-SMD_HD219F-3D05200
- added C1: 100nF, EasyEDA:C0603, F.Cu at (107.9, 57.5)
- added C2: 100nF, EasyEDA:C0603, F.Cu at (106.0, 57.4)
- added C3: 100uF, EasyEDA:CAP-SMD_BD6.3-L6.6-W6.6-LS7.2-R-RD, F.Cu at (118.2, 109.4)
- added U11: RT9742SNGV_C3235509, EasyEDA:SOT-23-3_L2.9-W1.6-P1.90-LS2.8-BR, F.Cu at (106.9, 54.2)
- added USB3: HDMI-101L, EasyEDA:HDMI-SMD_HDMI-101L, F.Cu at (101.1, 50.2)
- moved R8 77.6 mm to (128.9, 100.5)
- moved LED3 74.6 mm to (128.9, 98.6)
- moved R61 73.6 mm to (128.9, 102.4), turned to 0 degrees
- moved R6 71.7 mm to (121.8, 53.6), turned to -90 degrees
- moved LED5 71.0 mm to (127.4, 104.5), turned to 0 degrees
- moved U9 55.4 mm to (92.2, 110.7)
- moved R7 52.0 mm to (120.0, 53.6), turned to -90 degrees
- moved R69 49.0 mm to (91.8, 107.5)
- moved R60 48.6 mm to (95.8, 107.4), turned to 180 degrees
- moved R22 46.0 mm to (118.1, 53.7), turned to 90 degrees
- moved R70 45.7 mm to (95.8, 109.1)
- moved G*** 38.0 mm to (81.4, 57.0)
- moved R71 37.2 mm to (86.1, 110.4), turned to 180 degrees
- moved C18 14.7 mm to (65.4, 77.6), turned to -90 degrees
- moved R9 13.2 mm to (134.3, 90.8)
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Connections:
- CN5 pad 3: /CM5/USB2_N -> unconnected-(CN5-Pad3)
- CN5 pad 5: /CM5/USB2_P -> unconnected-(CN5-Pad5)
- CN5 pad 51: /CM5/HDMI0_CEC -> unconnected-(CN5-Pad51)
- CN5 pad 53: /CM5/HDMI0_HOTPLUG -> unconnected-(CN5-Pad53)
- FPC2 pad 13: /CM5/HDMI1_CEC -> GND
- R22 pad 1: GND -> /CM5/3.3V_CM5
Routing:
- net /CM5/3.3V_CM5: track 36.2 -> 222.8 mm, vias 4 -> 18
- net /CM5/5V: track 124.2 -> 250.5 mm, vias 48 -> 49
- net GND: track 28.2 -> 138.3 mm, vias 129 -> 429
- net /CM5/SD_DAT2: track 0.00 -> 73.4 mm, vias 0 -> 2
- net /CM5/SD_DAT3: track 0.00 -> 70.8 mm, vias 0 -> 2
- net /CM5/CAM_GPIO1: track 0.00 -> 67.4 mm, vias 0 -> 2
- net /CM5/CAM_GPIO0: track 0.00 -> 64.6 mm, vias 0 -> 2
- net /CM5/SD_CLK: track 0.00 -> 64.4 mm, vias 0 -> 2
- net /CM5/SD_CMD: track 0.00 -> 63.8 mm
- net /CM5/SDA1: track 0.00 -> 62.3 mm
- net /CM5/SD_DAT0: track 0.00 -> 62.0 mm, vias 0 -> 2
- net /CM5/PCM_DIN_SD: track 2.41 -> 63.5 mm, vias 1 -> 2
- net /CM5/SCL1: track 1.28 -> 62.0 mm, vias 1 -> 2
- net /CM5/SD_DAT1: track 0.00 -> 60.5 mm, vias 0 -> 2
- net /CM5/FAN_PWM: track 1.47 -> 61.2 mm, vias 1 -> 0
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Other:
- board size 80 x 105 mm -> 80.6 x 105 mm
- board text added: "C/D 0"
- board text added: "C/D 1"
- board text added: "LED_nACT"
- board text added: "nPWR_LED"
